File: Sensors_1.kicad_sch (KiCad schematic)
At the start: 25 parts, among them J7 Conn_01x06_Pin, J8 Conn_01x04_Pin, J9 Conn_01x02_Pin, U4 Ai-Thinker-Ra-01, U5 AT24C256, U6 Ai-Thinker-Ra-01SH

Commit message: feat: размешены все компоненты на печатной плате
Connections:
- net +3V3: now also C28.1, C29.1, C30.1, C31.1, C33.1, C34.1, DD1.6 (VDDIO), DD1.8 (VDD), R15.1, R16.1, R19.1, R20.1, U4.3 (VDD), U6.3 (VDD)
- net +3V3D: no longer C28.1, C29.1, C30.1, C31.1, C33.1, C34.1, DD1.6 (VDDIO), DD1.8 (VDD), R15.1, R16.1, R19.1, R20.1, U4.3 (VDD), U6.3 (VDD)
