File: External_interfaces.kicad_sch (KiCad schematic)
At the start: 42 parts, among them SW1 SW_Push, SW10 SW_Push, SW11 SW_Push, SW12 SW_Push, SW2 SW_Push, SW3 SW_Push, SW4 SW_Push, SW5 SW_Push, SW6 SW_Push, SW7 SW_Push, SW8 SW_Push, SW9 SW_Push

Commit message: feat: разведены линии DI большая часть
Connections:
- net DI6: now also C42.2, R36.1; no longer C43.2, R37.1
- net DI7: now also C43.2, R37.1; no longer C42.2, R36.1
Changed lines of the file:
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@@
+	)
+	(junction
+		(at 52.07 96.52)
+		(diameter 0)
+		(color 0 0 0 0)
 	)
 	(junction
@@
 	)
 	(junction
-		(at 52.07 96.52)
-		(diameter 0)
-		(color 0 0 0 0)
-	)
-	(junction
 		(at 130.81 107.95)
 		(diameter 0)
@@
 	(wire
 		(pts
+			(xy 205.74 72.39) (xy 212.09 72.39)
+		)
+		(stroke
+			(width 0)
+			(type default)
+		)
+	)
+	(wire
+		(pts
 			(xy 50.8 52.07) (xy 60.96 52.07)
 		)
@@
 	(wire
 		(pts
-			(xy 205.74 72.39) (xy 212.09 72.39)
+			(xy 44.45 96.52) (xy 52.07 96.52)
 		)
 		(stroke
@@
 		(pts
 			(xy 172.72 52.07) (xy 177.8 52.07)
-		)
-		(stroke
-			(width 0)
-			(type default)
-		)
-	)
-	(wire
-		(pts
-			(xy 43.18 96.52) (xy 52.07 96.52)
 		)
 		(stroke
@@
 	(global_label "DI7"
 		(shape input)
-		(at 43.18 96.52 180)
+		(at 205.74 72.39 180)
 		(fields_autoplaced yes)
 		(effects
@@
 		)
 		(property "Intersheetrefs" "${INTERSHEET_REFS}"
-			(at 37.1105 96.52 0)
+			(at 199.6705 72.39 0)
 			(hide yes)
 			(show_name no)
@@
 	(global_label "DI6"
 		(shape input)
-		(at 205.74 72.39 180)
+		(at 44.45 96.52 180)
 		(fields_autoplaced yes)
 		(effects
@@
 		)
 		(property "Intersheetrefs" "${INTERSHEET_REFS}"
-			(at 199.6705 72.39 0)
+			(at 38.3805 96.52 0)
 			(hide yes)
 			(show_name no)
